Commit message: imporved reset envirnoment in genesis

File: res/ur16e_robotiq.urdf (robot description, URDF)
Before this commit: robot ur16e, 24 links, 23 joints
Links:
- link base_link_inertia: geometry collision mesh filename=/home/yukun/Documents/RoboSkiAgent/temp/Universal_Robots_RO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; visual mesh filename=/home/yukun/Documents/RoboSkiAgent/temp/Universal_Robots_RO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
- link forearm_link: geometry collision mesh filename=/home/yukun/Documents/RoboSkiAgent/temp/Universal_Robots_RO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; visual mesh filename=/home/yukun/Documents/RoboSkiAgent/temp/Universal_Robots_RO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
- link left_inner_finger: geometry collision mesh filename=/home/yukun/Documents/RoboSkiAgent/temp/Robotiq-2f-85/robot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 scale=0.001 0.001 0.001; visual mesh filename=/home/yukun/Documents/RoboSkiAgent/temp/Robotiq-2f-85/robot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 scale=0.001 0.001 0.001
- link left_inner_knuckle: geometry collision mesh filename=/home/yukun/Documents/RoboSkiAgent/temp/Robotiq-2f-85/robot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 scale=0.001 0.001 0.001; visual mesh filename=/home/yukun/Documents/RoboSkiAgent/temp/Robotiq-2f-85/robot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 scale=0.001 0.001 0.001
- link left_outer_finger: geometry collision mesh filename=/home/yukun/Documents/RoboSkiAgent/temp/Robotiq-2f-85/robot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 scale=0.001 0.001 0.001; visual mesh filename=/home/yukun/Documents/RoboSkiAgent/temp/Robotiq-2f-85/robot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 scale=0.001 0.001 0.001
- link left_outer_knuckle: geometry collision mesh filename=/home/yukun/Documents/RoboSkiAgent/temp/Robotiq-2f-85/robot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 scale=0.001 0.001 0.001; visual mesh filename=/home/yukun/Documents/RoboSkiAgent/temp/Robotiq-2f-85/robot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 scale=0.001 0.001 0.001
- link right_inner_finger: geometry collision mesh filename=/home/yukun/Documents/RoboSkiAgent/temp/Robotiq-2f-85/robot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 scale=0.001 0.001 0.001; visual mesh filename=/home/yukun/Documents/RoboSkiAgent/temp/Robotiq-2f-85/robot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 scale=0.001 0.001 0.001
- link right_inner_knuckle: geometry collision mesh filename=/home/yukun/Documents/RoboSkiAgent/temp/Robotiq-2f-85/robot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 scale=0.001 0.001 0.001; visual mesh filename=/home/yukun/Documents/RoboSkiAgent/temp/Robotiq-2f-85/robot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 scale=0.001 0.001 0.001
- link right_outer_finger: geometry collision mesh filename=/home/yukun/Documents/RoboSkiAgent/temp/Robotiq-2f-85/robot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 scale=0.001 0.001 0.001; visual mesh filename=/home/yukun/Documents/RoboSkiAgent/temp/Robotiq-2f-85/robot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 scale=0.001 0.001 0.001
- link right_outer_knuckle: geometry collision mesh filename=/home/yukun/Documents/RoboSkiAgent/temp/Robotiq-2f-85/robot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 scale=0.001 0.001 0.001; visual mesh filename=/home/yukun/Documents/RoboSkiAgent/temp/Robotiq-2f-85/robot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 scale=0.001 0.001 0.001
- link robotiq_arg2f_base_link: geometry collision mesh filename=/home/yukun/Documents/RoboSkiAgent/temp/Robotiq-2f-85/robot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; visual mesh filename=/home/yukun/Documents/RoboSkiAgent/temp/Robotiq-2f-85/robot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 scale=0.001 0.001 0.001
- link shoulder_link: geometry collision mesh filename=/home/yukun/Documents/RoboSkiAgent/temp/Universal_Robots_RO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; visual mesh filename=/home/yukun/Documents/RoboSkiAgent/temp/Universal_Robots_RO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
- link upper_arm_link: geometry collision mesh filename=/home/yukun/Documents/RoboSkiAgent/temp/Universal_Robots_RO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; visual mesh filename=/home/yukun/Documents/RoboSkiAgent/temp/Universal_Robots_RO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
- link wrist_1_link: geometry collision mesh filename=/home/yukun/Documents/RoboSkiAgent/temp/Universal_Robots_RO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; visual mesh filename=/home/yukun/Documents/RoboSkiAgent/temp/Universal_Robots_RO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
- link wrist_2_link: geometry collision mesh filename=/home/yukun/Documents/RoboSkiAgent/temp/Universal_Robots_RO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; visual mesh filename=/home/yukun/Documents/RoboSkiAgent/temp/Universal_Robots_RO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
- link wrist_3_link: geometry collision mesh filename=/home/yukun/Documents/RoboSkiAgent/temp/Universal_Robots_RO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; visual mesh filename=/home/yukun/Documents/RoboSkiAgent/temp/Universal_Robots_RO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
Joints:
- joint left_inner_finger_joint: limit lower=0 upper=0.8757 effort=1000 velocity=2.0 -> lower=-0.8757 upper=0 effort=1000 velocity=2.0
- joint right_inner_finger_joint: limit lower=0 upper=0.8757 effort=1000 velocity=2.0 -> lower=-0.8757 upper=0 effort=1000 velocity=2.0

Commit message: auto snaping

File: res/ur16e_robotiq.urdf (robot description, URDF)
Before this commit: robot ur16e, 24 links, 23 joints
Links:
- link left_inner_finger: mass None -> 0.0104003125914103; geometry collision mesh filename=/home/yukun/Documents/RoboSkiAgent/temp/robotiq_2f_140_sour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; visual mesh filename=/home/yukun/Documents/RoboSkiAgent/temp/robotiq_2f_140_sour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
- link left_inner_finger_pad: geometry collision box size=0.03 0.07 0.0075; visual box size=0.027 0.065 0.0075
- link left_inner_knuckle: mass None -> 0.0271177346495152; geometry collision mesh filename=/home/yukun/Documents/RoboSkiAgent/temp/robotiq_2f_140_sour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; visual mesh filename=/home/yukun/Documents/RoboSkiAgent/temp/robotiq_2f_140_sour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
- link left_outer_finger: mass None -> 0.022614240507152; geometry collision mesh filename=/home/yukun/Documents/RoboSkiAgent/temp/robotiq_2f_140_sour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; visual mesh filename=/home/yukun/Documents/RoboSkiAgent/temp/robotiq_2f_140_sour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
- link left_outer_knuckle: mass None -> 0.00853198276973456; geometry collision mesh filename=/home/yukun/Documents/RoboSkiAgent/temp/robotiq_2f_140_sour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; visual mesh filename=/home/yukun/Documents/RoboSkiAgent/temp/robotiq_2f_140_sour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
- link right_inner_finger: mass None -> 0.0104003125914103; geometry collision mesh filename=/home/yukun/Documents/RoboSkiAgent/temp/robotiq_2f_140_sour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; visual mesh filename=/home/yukun/Documents/RoboSkiAgent/temp/robotiq_2f_140_sour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
- link right_inner_finger_pad: geometry collision box size=0.03 0.07 0.0075; visual box size=0.027 0.065 0.0075
- link right_inner_knuckle: mass None -> 0.0271177346495152; geometry collision mesh filename=/home/yukun/Documents/RoboSkiAgent/temp/robotiq_2f_140_sour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; visual mesh filename=/home/yukun/Documents/RoboSkiAgent/temp/robotiq_2f_140_sour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
- link right_outer_finger: mass None -> 0.022614240507152; geometry collision mesh filename=/home/yukun/Documents/RoboSkiAgent/temp/robotiq_2f_140_sour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; visual mesh filename=/home/yukun/Documents/RoboSkiAgent/temp/robotiq_2f_140_sour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
- link right_outer_knuckle: mass None -> 0.00853198276973456; geometry collision mesh filename=/home/yukun/Documents/RoboSkiAgent/temp/robotiq_2f_140_sour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; visual mesh filename=/home/yukun/Documents/RoboSkiAgent/temp/robotiq_2f_140_sour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
- link robotiq_arg2f_base_link: geometry collision mesh filename=/home/yukun/Documents/RoboSkiAgent/temp/robotiq_2f_140_sour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; visual mesh filename=/home/yukun/Documents/RoboSkiAgent/temp/robotiq_2f_140_sour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
Joints:
- joint finger_joint: axis 1 0 0 -> -1 0 0; limit lower=0 upper=0.8 effort=1000 velocity=2.0 -> lower=0 upper=0.7 effort=1000 velocity=2.0; origin xyz=0 -0.0306011 0.054904 rpy=0 0 3.141592653589793 -> xyz=0 -0.030601 0.054905 rpy=2.2957963267948966 0 0
- joint left_inner_finger_joint: limit lower=-0.8757 upper=0 effort=1000 velocity=2.0 -> lower=-0.8757 upper=0.8757 effort=1000 velocity=2.0; mimic joint=finger_joint multiplier=-1 offset=0 -> joint=finger_joint multiplier=1 offset=0; origin xyz=0 0.0061 0.0471 rpy=0 0 0 -> xyz=0 0.0817554015893473 -0.0282203446692936 rpy=-0.725 0 0
- joint left_inner_finger_pad_joint: origin xyz=0 -0.0220203446692936 0.03242 rpy=0 0 0 -> xyz=0 0.0457554015893473 -0.0272203446692936 rpy=0 0 0
- joint left_inner_knuckle_joint: limit lower=0 upper=0.8757 effort=1000 velocity=2.0 -> lower=-0.8757 upper=0.8757 effort=1000 velocity=2.0; mimic joint=finger_joint multiplier=1 offset=0 -> joint=finger_joint multiplier=-1 offset=0; origin xyz=0 -0.0127 0.06142 rpy=0 0 3.141592653589793 -> xyz=0 -0.0127 0.06142 rpy=2.2957963267948966 0 0.0
- joint left_outer_finger_joint: origin xyz=0 0.0315 -0.0041 rpy=0 0 0 -> xyz=0 0.01821998610742 0.0260018192872234 rpy=0 0 0
- joint right_inner_finger_joint: limit lower=-0.8757 upper=0 effort=1000 velocity=2.0 -> lower=-0.8757 upper=0.8757 effort=1000 velocity=2.0; mimic joint=finger_joint multiplier=-1 offset=0 -> joint=finger_joint multiplier=1 offset=0; origin xyz=0 0.0061 0.0471 rpy=0 0 0 -> xyz=0 0.0817554015893473 -0.0282203446692936 rpy=-0.725 0 0
- joint right_inner_finger_pad_joint: origin xyz=0 -0.0220203446692936 0.03242 rpy=0 0 0 -> xyz=0 0.0457554015893473 -0.0272203446692936 rpy=0 0 0
- joint right_inner_knuckle_joint: limit lower=0 upper=0.8757 effort=1000 velocity=2.0 -> lower=-0.8757 upper=0.8757 effort=1000 velocity=2.0; mimic joint=finger_joint multiplier=1 offset=0 -> joint=finger_joint multiplier=-1 offset=0; origin xyz=0 0.0127 0.06142 rpy=0 0 0.0 -> xyz=0 0.0127 0.06142 rpy=2.2957963267948966 0 -3.141592653589793
- joint right_outer_finger_joint: origin xyz=0 0.0315 -0.0041 rpy=0 0 0 -> xyz=0 0.01821998610742 0.0260018192872234 rpy=0 0 0
- joint right_outer_knuckle_joint: limit lower=0 upper=0.81 effort=1000 velocity=2.0 -> lower=-0.725 upper=0.725 effort=1000 velocity=2.0; mimic joint=finger_joint multiplier=1 offset=0 -> joint=finger_joint multiplier=-1 offset=0; origin xyz=0 0.0306011 0.054904 rpy=0 0 0 -> xyz=0 0.030601 0.054905 rpy=2.2957963267948966 0 3.141592653589793
