Commit message: res

File: res/ur16e_raw.urdf (robot description, URDF)
Before this commit: robot ur16e, 13 links, 12 joints
Links:
- link base_link_inertia: geometry collision mesh filename=robot_models/Universal_Robots_ROS2_Description/meshes/ur10e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; visual mesh filename=robot_models/Universal_Robots_ROS2_Description/meshes/ur10e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
- link forearm_link: geometry collision mesh filename=robot_models/Universal_Robots_ROS2_Description/meshes/ur16e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; visual mesh filename=robot_models/Universal_Robots_ROS2_Description/meshes/ur16e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
- link shoulder_link: geometry collision mesh filename=robot_models/Universal_Robots_ROS2_Description/meshes/ur10e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; visual mesh filename=robot_models/Universal_Robots_ROS2_Description/meshes/ur10e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
- link upper_arm_link: geometry collision mesh filename=robot_models/Universal_Robots_ROS2_Description/meshes/ur16e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; visual mesh filename=robot_models/Universal_Robots_ROS2_Description/meshes/ur16e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
- link wrist_1_link: geometry collision mesh filename=robot_models/Universal_Robots_ROS2_Description/meshes/ur10e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; visual mesh filename=robot_models/Universal_Robots_ROS2_Description/meshes/ur10e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
- link wrist_2_link: geometry collision mesh filename=robot_models/Universal_Robots_ROS2_Description/meshes/ur10e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; visual mesh filename=robot_models/Universal_Robots_ROS2_Description/meshes/ur10e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
- link wrist_3_link: geometry collision mesh filename=robot_models/Universal_Robots_ROS2_Description/meshes/ur10e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; visual mesh filename=robot_models/Universal_Robots_ROS2_Description/meshes/ur10e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

File: res/ur16e_robotiq.urdf (robot description, URDF)
Before this commit: robot ur16e, 24 links, 23 joints
Links:
- link base_link_inertia: geometry collision mesh filename=robot_models/Universal_Robots_ROS2_Description/meshes/ur10e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; visual mesh filename=robot_models/Universal_Robots_ROS2_Description/meshes/ur10e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
- link forearm_link: geometry collision mesh filename=robot_models/Universal_Robots_ROS2_Description/meshes/ur16e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; visual mesh filename=robot_models/Universal_Robots_ROS2_Description/meshes/ur16e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
- link left_inner_finger: geometry collision mesh filename=robot_models/robotiq_2f_140_gripper_visualization/meshes/co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; visual mesh filename=robot_models/robotiq_2f_140_gripper_visualization/meshes/vi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
- link left_inner_knuckle: geometry collision mesh filename=robot_models/robotiq_2f_140_gripper_visualization/meshes/co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; visual mesh filename=robot_models/robotiq_2f_140_gripper_visualization/meshes/vi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
- link left_outer_finger: geometry collision mesh filename=robot_models/robotiq_2f_140_gripper_visualization/meshes/co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; visual mesh filename=robot_models/robotiq_2f_140_gripper_visualization/meshes/vi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
- link left_outer_knuckle: geometry collision mesh filename=robot_models/robotiq_2f_140_gripper_visualization/meshes/co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; visual mesh filename=robot_models/robotiq_2f_140_gripper_visualization/meshes/vi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
- link right_inner_finger: geometry collision mesh filename=robot_models/robotiq_2f_140_gripper_visualization/meshes/co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; visual mesh filename=robot_models/robotiq_2f_140_gripper_visualization/meshes/vi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
- link right_inner_knuckle: geometry collision mesh filename=robot_models/robotiq_2f_140_gripper_visualization/meshes/co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; visual mesh filename=robot_models/robotiq_2f_140_gripper_visualization/meshes/vi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
- link right_outer_finger: geometry collision mesh filename=robot_models/robotiq_2f_140_gripper_visualization/meshes/co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; visual mesh filename=robot_models/robotiq_2f_140_gripper_visualization/meshes/vi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
- link right_outer_knuckle: geometry collision mesh filename=robot_models/robotiq_2f_140_gripper_visualization/meshes/co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; visual mesh filename=robot_models/robotiq_2f_140_gripper_visualization/meshes/vi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
- link robotiq_arg2f_base_link: geometry collision mesh filename=robot_models/robotiq_2f_140_gripper_visualization/meshes/co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; visual mesh filename=robot_models/robotiq_2f_140_gripper_visualization/meshes/vi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
- link shoulder_link: geometry collision mesh filename=robot_models/Universal_Robots_ROS2_Description/meshes/ur10e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; visual mesh filename=robot_models/Universal_Robots_ROS2_Description/meshes/ur10e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
- link upper_arm_link: geometry collision mesh filename=robot_models/Universal_Robots_ROS2_Description/meshes/ur16e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; visual mesh filename=robot_models/Universal_Robots_ROS2_Description/meshes/ur16e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
- link wrist_1_link: geometry collision mesh filename=robot_models/Universal_Robots_ROS2_Description/meshes/ur10e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; visual mesh filename=robot_models/Universal_Robots_ROS2_Description/meshes/ur10e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
- link wrist_2_link: geometry collision mesh filename=robot_models/Universal_Robots_ROS2_Description/meshes/ur10e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; visual mesh filename=robot_models/Universal_Robots_ROS2_Description/meshes/ur10e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
- link wrist_3_link: geometry collision mesh filename=robot_models/Universal_Robots_ROS2_Description/meshes/ur10e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; visual mesh filename=robot_models/Universal_Robots_ROS2_Description/meshes/ur10e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
